File: hardware/shutter-tester.kicad_pcb (KiCad board)
At the start: 2 copper layers, 50 x 34 mm, 18 parts, among them J1 Conn_01x05_Pin, U1 ESP32-C3_SUPERMINI, U2 Sensor-1, U3 Sensor-3, U4 Sensor-2

Commit message: fix: groundplane issue w/ 2 via in PCB; update pictures
Routing:
- net GND: vias 1 -> 3
Other:
- board text added: "v1.1 2025-01-27"
- board text removed: "v1.0 2024-12-31"
Changed lines of the file:
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@@
 			(usegerberattributes yes)
 			(usegerberadvancedattributes yes)
-			(creategerberjobfile yes)
+			(creategerberjobfile no)
 			(dashed_line_dash_ratio 12.000000)
 			(dashed_line_gap_ratio 3.000000)
@@
 			(plotinvisibletext no)
 			(sketchpadsonfab no)
-			(subtractmaskfromsilk no)
+			(subtractmaskfromsilk yes)
 			(outputformat 1)
 			(mirror no)
 			(drillshape 0)
 			(scaleselection 1)
-			(outputdirectory "output/v1.0/")
+			(outputdirectory "output/v1.1/")
 		)
 	)
@@
 		(tags "capacitor handsolder")
 		(property "Reference" "C3"
-			(at -3.556 0 360)
+			(at -3.556 0 0)
 			(layer "F.SilkS")
 			(effects
@@
 		)
 		(property "Value" "C"
-			(at 1.524 -1.778 360)
+			(at 1.524 -1.778 0)
 			(layer "F.Fab")
 			(effects
@@
 		)
 		(fp_text user "${REFERENCE}"
-			(at 0 0 360)
+			(at 0 0 0)
 			(layer "F.Fab")
 			(effects
@@
 		)
 		(property "Value" "C"
-			(at -3.048 0 360)
+			(at -3.048 0 0)
 			(layer "F.Fab")
 			(effects
@@
 		)
 		(fp_text user "${REFERENCE}"
-			(at 3.302 0 360)
+			(at 3.302 0 0)
 			(layer "F.Fab")
 			(effects
@@
 		(tags "capacitor handsolder")
 		(property "Reference" "C1"
-			(at 3.302 0 360)
+			(at 3.302 0 0)
 			(layer "F.SilkS")
 			(effects
@@
 		)
 		(property "Value" "C"
-			(at -3.302 0 360)
+			(at -3.302 0 0)
 			(layer "F.Fab")
 			(effects
@@
 		)
 		(fp_text user "${REFERENCE}"
-			(at 0 0 360)
+			(at 0 0 0)
 			(layer "F.Fab")
 			(effects
@@
 		)
 	)
-	(gr_text "v1.0 2024-12-31"
+	(gr_text "v1.1 2025-01-27"
 		(at 79.502 115.824 0)
 		(layer "F.SilkS")
@@
 		(net 2)
 	)
+	(via
+		(at 112.63 105.092)
+		(size 0.6)
+		(drill 0.3)
+		(layers "F.Cu" "B.Cu")
+		(free yes)
+		(net 2)
+	)
+	(via
+		(at 90.13 104.592)
+		(size 0.6)
+		(drill 0.3)
+		(layers "F.Cu" "B.Cu")
+		(free yes)
+		(net 2)
+	)
