File: hardware/shutter-tester.kicad_pcb (KiCad board)
At the start: 2 copper layers, 50 x 34 mm, 18 parts, among them J1 Conn_01x05_Pin, U1 ESP32-C3_SUPERMINI, U2 Sensor-1, U3 Sensor-3, U4 Sensor-2

Commit message: v2.0 of the hardware
Parts:
- removed J1: Conn_01x05_Pin, Connector_PinHeader_2.54mm:PinHeader_1x05_P2.54mm_Vertical
- removed REF**: OSHW-Logo2_7.3x6mm_SilkScreen, Symbol:OSHW-Logo2_7.3x6mm_SilkScreen
- C1, C2, C3: value C -> 0.01uF
- R4, R6, R8: value 2k -> 1k
- R5, R7, R9: value 1k -> 2k
- moved R7 13.7 mm to (94.2, 93.2)
- moved R6 8.99 mm to (91.4, 93.2), turned to -90 degrees
- moved C1 8.38 mm to (97.5, 114.0), turned to 0 degrees
- moved R9 6.36 mm to (102.6, 93.2)
- moved R2 5.95 mm to (88.6, 93.2)
- moved C2 5.24 mm to (87.4, 100.1), turned to -90 degrees
- moved R3 4.83 mm to (97.0, 93.2)
- moved R8 0.80 mm to (99.8, 93.2)
- moved C3 0.49 mm to (113.9, 85.9)
Connections:
- C1 pad 2: Net-(U2-OUT) -> +5V
- C2 pad 1: GND -> +5V
- C2 pad 2: Net-(U4-OUT) -> GND
- C3 pad 2: Net-(U3-OUT) -> +5V
- U1 pad 0: unconnected-(U1-GPIO0-Pad0) -> SENSOR_1
- U1 pad 2: SENSOR_1 -> unconnected-(U1-GPIO2-Pad2)
- U1 pad 20: unconnected-(U1-GPIO20-Pad20) -> SENSOR_3
- U1 pad 21: unconnected-(U1-GPIO21-Pad21) -> SENSOR_2
- U1 pad 3: SENSOR_2 -> unconnected-(U1-GPIO3-Pad3)
- U1 pad 4: SENSOR_3 -> unconnected-(U1-GPIO4-Pad4)
Routing:
- net SENSOR_2: track 64.9 -> 18.5 mm, vias 2 -> 0
- net SENSOR_3: track 41.5 -> 11.0 mm
- net SENSOR_1: track 38.4 -> 9.47 mm, vias 2 -> 0
- net +5V: track 113.6 -> 102.5 mm, vias 4 -> 0
- net Net-(U3-OUT): track 20.9 -> 13.3 mm
- net Net-(U2-OUT): track 10.7 -> 7.84 mm
- net GND: track 3.13 -> 0.25 mm, vias 1 -> 0
- net Net-(U4-OUT): track 11.8 -> 13.8 mm
Other:
- outline, holes or cut-outs redrawn
- board text added: "v2.0 2025-01-25"
- board text removed: "v1.0 2024-12-31"

Commit message: Don't use GPIO 0 for sensor input
Connections:
- U1 pad 0: SENSOR_1 -> unconnected-(U1-GPIO0-Pad0)
- U1 pad 1: unconnected-(U1-GPIO1-Pad1) -> SENSOR_1
Routing:
- net SENSOR_1: track 9.47 -> 12.6 mm
Other:
- board text added: "v2.1 2025-01-25"
- board text removed: "v2.0 2025-01-25"
Changed lines of the file:
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@@
 			(drillshape 0)
 			(scaleselection 1)
-			(outputdirectory "output/v2.0/")
+			(outputdirectory "output/v2.1/")
 		)
 	)
@@
 	(net 11 "unconnected-(U1-GPIO4-Pad4)")
 	(net 12 "unconnected-(U1-GPIO8-Pad8)")
-	(net 13 "unconnected-(U1-GPIO1-Pad1)")
+	(net 13 "unconnected-(U1-GPIO0-Pad0)")
 	(net 14 "unconnected-(U1-GPIO2-Pad2)")
 	(net 15 "unconnected-(U1-3V3-Pad3.3)")
@@
 		)
 		(property "Value" "1k"
-			(at -3.048 0 360)
+			(at -3.048 0 0)
 			(layer "F.SilkS")
 			(effects
@@
 		(tags "capacitor handsolder")
 		(property "Reference" "C3"
-			(at -3.556 0 360)
+			(at -3.556 0 0)
 			(layer "F.SilkS")
 			(effects
@@
 		)
 		(property "Value" "0.01uF"
-			(at 1.524 -1.778 360)
+			(at 1.524 -1.778 0)
 			(layer "F.Fab")
 			(effects
@@
 		)
 		(fp_text user "${REFERENCE}"
-			(at 0 0 360)
+			(at 0 0 0)
 			(layer "F.Fab")
 			(effects
@@
 		)
 		(property "Value" "1k"
-			(at -3.074 0 360)
+			(at -3.074 0 0)
 			(layer "F.SilkS")
 			(effects
@@
 		)
 		(property "Value" "Sensor-1"
-			(at -2.05 -1.09 360)
+			(at -2.05 -1.09 0)
 			(layer "F.SilkS")
 			(effects
@@
 			(size 1.905 1.905)
 			(layers "F.Cu" "F.Paste" "F.Mask")
-			(net 1 "SENSOR_1")
+			(net 13 "unconnected-(U1-GPIO0-Pad0)")
 			(pinfunction "GPIO0")
 			(pintype "bidirectional")
@@
 			(size 1.905 1.905)
 			(layers "F.Cu" "F.Paste" "F.Mask")
-			(net 13 "unconnected-(U1-GPIO1-Pad1)")
+			(net 1 "SENSOR_1")
 			(pinfunction "GPIO1")
 			(pintype "bidirectional")
@@
 		(tags "capacitor handsolder")
 		(property "Reference" "C1"
-			(at 3.302 0 360)
+			(at 3.302 0 0)
 			(layer "F.SilkS")
 			(effects
@@
 		)
 		(property "Value" "0.01uF"
-			(at -3.302 0 360)
+			(at -3.302 0 0)
 			(layer "F.Fab")
 			(effects
@@
 		)
 		(fp_text user "${REFERENCE}"
-			(at 0 0 360)
+			(at 0 0 0)
 			(layer "F.Fab")
 			(effects
@@
 		(layer "Edge.Cuts")
 	)
-	(gr_text "v2.0 2025-01-25"
+	(gr_text "v2.1 2025-01-25"
 		(at 81.534 91.186 90)
 		(layer "B.SilkS")
@@
 	)
 	(segment
+		(start 102.463 112.141)
+		(end 109.855 112.141)
+		(width 0.3)
+		(layer "F.Cu")
+		(net 1)
+	)
+	(segment
 		(start 99.06 111.532)
 		(end 101.854 111.532)
@@
 	)
 	(segment
-		(start 102.134 111.532)
-		(end 104.14 113.538)
+		(start 110.236 112.522)
+		(end 110.236 113.538)
 		(width 0.3)
 		(layer "F.Cu")
@@
 	)
 	(segment
-		(start 101.854 111.532)
-		(end 102.134 111.532)
+		(start 109.855 112.141)
+		(end 110.236 112.522)
 		(width 0.3)
 		(layer "F.Cu")
@@
 	)
 	(segment
-		(start 104.14 113.538)
-		(end 107.696 113.538)
+		(start 101.854 111.532)
+		(end 102.463 112.141)
 		(width 0.3)
 		(layer "F.Cu")
